File: PCB/LEDPanelKit.kicad_pcb (KiCad board)
At the start: 2 copper layers, 96 x 128 mm, 52 parts, among them J1 Conn_01x02_RESET, J2 Conn_01x04_Debug, J3 Conn_01x05_POWER_IN, J4 Screw_Terminal_01x02, J5 Screw_Terminal_01x02, SW1 Rotary_Encoder_Switch, SW2 SW_Push, U1 ESP32_DEVKITC, U10 microSD_SPI_Module, U2 SEEED_GROVE, U3 MPU-6500_Module, U4 GY-BMP_E280, U5 RTC_PCF8563module, U6 ESP32_DEVKIT_V1, U7 LM386Module_Taobao, U8 HUB75, U9 LicheePiNano_1.27

Commit message: Beta1 PCB
Parts:
- removed the REF** at (131.0, 41.0)
- removed the REF** at (132.0, 122.0)
- removed the REF** at (198.0, 119.5)
- removed the REF** at (155.0, 117.0)
- removed the REF** at (216.0, 59.5)
- added C3: 330uF, Capacitor_THT:CP_Radial_D8.0mm_P5.00mm, F.Cu at (149.6, 46.2)
- added D1: LED, LED_THT:LED_D5.0mm, F.Cu at (194.5, 3.50)
- added G***: LOGO, library:LovyanGFX-Logo-20mm, F.Cu at (220.3, 18.5)
- added G***: LOGO, library:AVTOKYO-SHOOT-2-size2, F.Cu at (217.5, 84.0)
- added G***: LOGO, library:AVTOKYO-SHOOT-1-size2, F.Cu at (217.5, 113.0)
- added G***: LOGO, library:AVTOKYO-SHOOT-3-size2, F.Cu at (217.2, 73.8)
- added G***: LOGO, library:AVTOKYO-SHOOT-2-size2, F.Cu at (217.5, 104.2)
- added G***: LOGO, library:AVTOKYO-COPY-20mm, F.Cu at (186.5, 18.5)
- added G***: LOGO, library:LOWLEVEL_LOGO_9mm, F.Cu at (188.5, 26.2)
- added G***: LOGO, library:AKBROBOT_LOGO_9mm, F.Cu at (142.5, 102.8)
- added JP3: Jumper, Connector_PinHeader_2.54mm:PinHeader_1x02_P2.54mm_Vertical, F.Cu at (203.0, 107.5)
- added JP4: Jumper_NC_Dual, Jumper:SolderJumper-3_P1.3mm_Bridged12_Pad1.0x1.5mm, F.Cu at (132.5, 92.7)
- added JP5: Jumper, Jumper:SolderJumper-2_P1.3mm_Open_TrianglePad1.0x1.5mm, F.Cu at (131.7, 79.7)
- added OSHW: 1.1, library:OSHW_LOGL_SYLK_5mm, F.Cu at (211.5, 73.2)
- added OSHW: 1.1, library:OSHW_LOGL_SYLK_5mm, F.Cu at (211.5, 67.2)
- added OSHW: 1.1, library:OSHW_LOGL_SYLK_5mm, F.Cu at (217.2, 67.2)
- R2: value 330 -> 10k
- U10: moved to B.Cu
- moved REF** 89.8 mm to (205.0, 2.00)
- moved U10 78.8 mm to (206.5, 20.0), turned to 0 degrees
- moved R2 45.7 mm to (180.0, 13.6), turned to 90 degrees
- moved U7 45.4 mm to (181.0, 86.0), turned to 270 degrees
- moved LS1 44.4 mm to (199.0, 85.0)
- moved J5 39.8 mm to (133.0, 67.2), turned to 270 degrees
- moved U6 37.6 mm to (185.6, 48.3)
- moved J4 37.3 mm to (133.0, 53.8), turned to 270 degrees
- moved C1 37.1 mm to (179.4, 26.2), turned to 180 degrees
- moved C2 37.0 mm to (179.5, 23.2)
- moved R1 36.9 mm to (202.0, 2.00), turned to 180 degrees
- moved U1 35.8 mm to (190.7, 45.1)
- moved U8 29.3 mm to (141.0, 56.4), turned to 0 degrees
- moved G*** 25.5 mm to (184.5, 114.5), turned to 180 degrees
- moved REF** 24.2 mm to (190.0, 3.50)
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Connections:
- net /LEDA0 renamed /LEDA
- net /LEDA1 renamed /LEDB
- net /LEDA2 renamed /LEDC
- net /LEDA3 renamed /LEDD
- BZ1 pad 1: /BUZZER -> Net-(BZ1-Pad1)
- C2 pad 1: Net-(C2-Pad1) -> /SW_B
- C2 pad 2: Net-(C2-Pad2) -> /SW_A
- R1 pad 1: /SW_A -> /LEDE_BUZZER
- R1 pad 2: Net-(C2-Pad2) -> Net-(D1-Pad2)
- R2 pad 1: /SW_B -> /SW_ANALOG
- R2 pad 2: Net-(C2-Pad1) -> Net-(R2-Pad2)
- R5 pad 1: /SW_ANALOG -> +3V3
- R5 pad 2: Net-(R5-Pad2) -> /SW_B
- R6 pad 1: +3V3 -> /LEDE_BUZZER
- R6 pad 2: /SW_B -> GND
- SW1 pad A: Net-(C2-Pad1) -> /SW_B
- SW1 pad B: Net-(C2-Pad2) -> /SW_A
- SW1 pad S1: /SW_ANALOG -> Net-(R2-Pad2)
- SW2 pad 2: Net-(R5-Pad2) -> /SW_ANALOG
- U1 pad 24: /BUZZER -> /LEDE_BUZZER
- U2 pad 1: /SCL -> /I2C_SCL
- U2 pad 2: /SDA -> /I2C_SDA
- U2 pad 3: +3V3 -> Net-(JP4-Pad2)
- U3 pad 3: /SCL -> /I2C_SCL
- U3 pad 4: /SDA -> /I2C_SDA
- U4 pad 3: /SCL -> /I2C_SCL
- U4 pad 4: /SDA -> /I2C_SDA
- U5 pad 3: /SCL -> /I2C_SCL
- U5 pad 4: /SDA -> /I2C_SDA
- U6 pad 19: /BUZZER -> /LEDE_BUZZER
- U8 pad 8: GND -> Net-(JP5-Pad2)
Routing:
- net /LEDE_BUZZER: track 0.00 -> 265.6 mm, vias 0 -> 6
- net /I2C_SDA: track 5.08 -> 145.1 mm
- net /I2C_SCL: track 5.08 -> 141.1 mm
- net /SCL: track 97.2 -> 0.00 mm, vias 1 -> 0
- net Net-(C2-Pad1): track 92.9 -> 0.00 mm, vias 1 -> 0
- net /SDA: track 81.0 -> 0.00 mm, vias 2 -> 0
- net Net-(C2-Pad2): track 79.1 -> 0.00 mm, vias 1 -> 0
- net /SDMOSI_SMISO_TX2: track 205.2 -> 127.7 mm, vias 5 -> 2
- net /SW_ANALOG: track 127.8 -> 69.5 mm, vias 3 -> 1
- net /SDMISO_SMOSI_RX2: track 177.5 -> 122.2 mm, vias 4 -> 3
- net Net-(J2-Pad1): track 114.9 -> 69.1 mm
- net /BUZZER: track 41.4 -> 0.00 mm
- net /TX: track 124.8 -> 85.7 mm, vias 1 -> 2
- net /LEDG1: track 47.0 -> 80.3 mm, vias 1 -> 2
- net /LEDB1: track 46.2 -> 79.0 mm, vias 2 -> 1
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Other:
- outline, holes or cut-outs redrawn
- board text added: "(331)"
- board text added: "10kΩ(104)x4"
- board text added: "330Ω"
- board text added: "5V 3.3V"
- board text added: "AKBONE2022"
- board text added: "AKBONE2022 Beta1"
- board text added: "B B W G RED"
- board text added: "BUZZER ON/OFF"
- board text added: "DABO"
- board text added: "GND VCC SDA SCL"
- board text added: "HY2.0-4P VCC SELECT"
- board text added: "I2C"
- board text added: "If use 128x64 panel, Please SHORT(JP5) and buzzer OFF(JP3)"
- board text added: "Lichee UART to ESP32 UART1or2"
- board text added: "Linux 3.3V"
- board text added: "Micro SD Module Caution! Turn over and attach."
- board text added: "NAME"
- board text added: "Please OFF"
- board text added: "when 128 x 64 panel,"
- board text removed: "104 x 4"
- board text removed: "3.3V"
- board text removed: "331 x 2"
- board text removed: "AKBONE 2022"
- board text removed: "GROVE"
- board text removed: "Lichee UART to ESP32 UART1 or 2"
