File: PCB/LEDPanelKit.sch (KiCad schematic (older format))
At the start: 29 parts, among them J1 Conn_01x02_RESET, J2 Conn_01x04_Debug, J3 Conn_01x05_POWER_IN, J4 Screw_Terminal_01x02, J5 Screw_Terminal_01x02, SW1 Rotary_Encoder_Switch, SW2 SW_Push, U1 ESP32_DEVKITC, U10 microSD_SPI_Module, U2 SEEED_GROVE, U3 MPU-6500_Module, U4 GY-BMP_E280, U5 RTC_PCF8563module, U6 ESP32_DEVKIT_V1, U7 LM386Module_Taobao, U8 HUB75, U9 LicheePiNano_1.27

Commit message: Beta1 PCB
Parts:
- removed R2: 330, Resistor_SMD:R_1206_3216Metric_Pad1.30x1.75mm_HandSolder, symbol Device:R
- added C3: 330uF, Capacitor_THT:CP_Radial_D8.0mm_P5.00mm, symbol Device:CP
- added D1: LED, LED_THT:LED_D5.0mm, symbol Device:LED
- added JP3: Jumper, Connector_PinHeader_2.54mm:PinHeader_1x02_P2.54mm_Vertical, symbol Device:Jumper
- added JP4: Jumper_NC_Dual, Jumper:SolderJumper-3_P1.3mm_Bridged12_Pad1.0x1.5mm, symbol Device:Jumper_NC_Dual
- added JP5: Jumper, Jumper:SolderJumper-2_P1.3mm_Open_TrianglePad1.0x1.5mm, symbol Device:Jumper
- added R6: 10k, Resistor_SMD:R_1206_3216Metric_Pad1.30x1.75mm_HandSolder, symbol Device:R
- renumbered R5 to R2, R6 to R5
Connections:
- net SCL is gone; now on net I2C_SCL: U2.1 (Yellow/Dn/An/RX/SCL), U3.3 (SCL), U4.3 (SCL), U5.3 (SCL)
- net SDA is gone; now on net I2C_SDA: U2.2 (White/Dn1/An1/TX/SDA), U3.4 (SDA), U4.4 (SDA), U5.4 (SDA)
- net +3V3: now also JP4.1; no longer U2.3 (Red/VCC)
- net +5V: now also C3.1, JP4.3
- net GND: now also C3.2, D1.1 (K), R6.2; no longer U8.8 (GND/E)
- net SW_A: now also C2.2, SW1.B; no longer R1.1
- net SW_ANALOG: now also SW2.2; no longer SW1.S1
- net SW_B: now also C2.1, SW1.A
- net at R2.2: now also SW1.S1; no longer SW2.2
- net BUZZER renamed LEDE_BUZZER
- net LEDE_BUZZER: now also R1.1, JP3.1, JP5.1, R6.1; no longer BZ1.1 (-)
- net LEDA0 renamed LEDA
- net LEDA1 renamed LEDB
- net LEDA2 renamed LEDC
- net LEDA3 renamed LEDD
- new net: BZ1.1 (-), JP3.2
- new net: JP4.2, U2.3 (Red/VCC)
- new net: JP5.2, U8.8 (GND/E)
- new net: D1.2 (A), R1.2
Other:
- moved on the sheet: BZ1, R1, R2, U10, U2, U3, U4, U5
